File: PCB/KiCad_Saim-Chan/SAIM-Chan.kicad_sch (KiCad schematic)
At the start: 155 parts, among them J1 Conn_01x02, J2 Conn_01x02, SW1 SW_SPDT_312, SW2 SW_SPDT_312, SW3 Switch, SW4 Switch, U1 Nice_Nano_V2, U2 Nice_Nano_V2

Commit message: Update
Parts:
- S1, S10, S11, S12, S13, S16, S17, S18, S19, S2, S20, S21, S22, S23, S24, S25, S26, S27, S3, S30, S31, S32, S33, S34, S35, S36, S37, S38, S39, S4, S40, S43, S44, S45, S46, S47, S48, S49, S5, S50, S51, S52, S54, S55, S56, S57, S58, S6, S61, S62, S63, S64, S65, S7, S8, S9: footprint Switches:Hotswap_Choc_V1_1.00u -> ScottoKeebs_Hotswap:Hotswap_Choc_V1_1.00u
- S14, S29, S53: footprint Switches:Hotswap_Choc_V1_1.50u -> ScottoKeebs_Hotswap:Hotswap_Choc_V1_1.50u
- S15, S28: footprint Switches:Hotswap_Choc_V1_1.25u -> ScottoKeebs_Hotswap:Hotswap_Choc_V1_1.25u
- S41, S42: footprint Switches:Hotswap_Choc_V1_1.75u -> ScottoKeebs_Hotswap:Hotswap_Choc_V1_1.75u
- S59, S60: footprint Switches:Hotswap_Choc_V1_3.00u -> ScottoKeebs_Hotswap:Hotswap_Choc_V1_3.00u

Commit message: Update
Parts:
- D1, D10, D11, D12, D13, D14, D15, D16, D17, D18, D19, D2, D20, D21, D22, D23, D24, D25, D26, D27, D28, D29, D3, D30, D31, D32, D33, D34, D35, D36, D37, D38, D39, D4, D40, D41, D42, D43, D44, D45, D46, D47, D48, D49, D5, D50, D51, D52, D53, D54, D55, D56, D57, D58, D59, D6, D60, D61, D62, D63, D64, D65, D7, D8, D9: value ~ -> (none); footprint ScottoKeebs_Components:Diode_SOD-123 -> Diodes:Diode_SOD-123
- Display_1, Display_2: footprint ScottoKeebs_Components:OLED_128x32 -> OLED_128x32:OLED_128x32
- S1, S10, S11, S12, S13, S16, S17, S18, S19, S2, S20, S21, S22, S23, S24, S25, S26, S27, S3, S30, S31, S32, S33, S34, S35, S36, S37, S38, S39, S4, S40, S43, S44, S45, S46, S47, S48, S49, S5, S50, S51, S52, S54, S55, S56, S57, S58, S6, S61, S62, S63, S64, S65, S7, S8, S9: value ~ -> (none); footprint ScottoKeebs_Hotswap:Hotswap_Choc_V1_1.00u -> Switches:Hotswap_Choc_V1_1.00u
- S14, S29, S53: value ~ -> (none); footprint ScottoKeebs_Hotswap:Hotswap_Choc_V1_1.50u -> Switches:Hotswap_Choc_V1_1.50u
- S15, S28: value ~ -> (none); footprint ScottoKeebs_Hotswap:Hotswap_Choc_V1_1.25u -> Switches:Hotswap_Choc_V1_1.25u
- S41, S42: value ~ -> (none); footprint ScottoKeebs_Hotswap:Hotswap_Choc_V1_1.75u -> Switches:Hotswap_Choc_V1_1.75u
- S59, S60: value ~ -> (none); footprint ScottoKeebs_Hotswap:Hotswap_Choc_V1_3.00u -> Switches:Hotswap_Choc_V1_3.00u
- U1, U2: footprint ScottoKeebs_MCU:Nice_Nano_V2 -> Nice_Nano_v2:Nice_Nano_V2

Commit message: Update
Parts:
- D1, D10, D11, D12, D13, D14, D15, D16, D17, D18, D19, D2, D20, D21, D22, D23, D24, D25, D26, D27, D28, D29, D3, D30, D31, D32, D33, D34, D35, D36, D37, D38, D39, D4, D40, D41, D42, D43, D44, D45, D46, D47, D48, D49, D5, D50, D51, D52, D53, D54, D55, D56, D57, D58, D59, D6, D60, D61, D62, D63, D64, D65, D7, D8, D9: footprint Diodes:Diode_SOD-123 -> ScottoKeebs_Components:Diode_SOD-123
- Display_1, Display_2: footprint OLED_128x32:OLED_128x32 -> ScottoKeebs_Components:OLED_128x32
- S1, S10, S11, S12, S13, S16, S17, S18, S19, S2, S20, S21, S22, S23, S24, S25, S26, S27, S3, S30, S31, S32, S33, S34, S35, S36, S37, S38, S39, S4, S40, S43, S44, S45, S46, S47, S48, S49, S5, S50, S51, S52, S54, S55, S56, S57, S58, S6, S61, S62, S63, S64, S65, S7, S8, S9: footprint Switches:Hotswap_Choc_V1_1.00u -> ScottoKeebs_Hotswap:Hotswap_Choc_V1_1.00u
- S14, S29, S53: footprint Switches:Hotswap_Choc_V1_1.50u -> ScottoKeebs_Hotswap:Hotswap_Choc_V1_1.50u
- S15, S28: footprint Switches:Hotswap_Choc_V1_1.25u -> ScottoKeebs_Hotswap:Hotswap_Choc_V1_1.25u
- S41, S42: footprint Switches:Hotswap_Choc_V1_1.75u -> ScottoKeebs_Hotswap:Hotswap_Choc_V1_1.75u
- S59, S60: footprint Switches:Hotswap_Choc_V1_3.00u -> ScottoKeebs_Hotswap:Hotswap_Choc_V1_3.00u
- U1, U2: footprint Nice_Nano_v2:Nice_Nano_V2 -> ScottoKeebs_MCU:Nice_Nano_V2

Commit message: Update
Parts:
- S1, S10, S11, S12, S13, S16, S17, S18, S19, S2, S20, S21, S22, S23, S24, S25, S26, S27, S3, S30, S31, S32, S33, S34, S35, S36, S37, S38, S39, S4, S40, S43, S44, S45, S46, S47, S48, S49, S5, S50, S51, S52, S54, S55, S56, S57, S58, S6, S61, S62, S63, S64, S65, S7, S8, S9: footprint ScottoKeebs_Hotswap:Hotswap_Choc_V1_1.00u -> With-Hotswap & Switches:Hotswap_Choc_V1_1.00u
- S14, S29, S53: footprint ScottoKeebs_Hotswap:Hotswap_Choc_V1_1.50u -> With-Hotswap & Switches:Hotswap_Choc_V1_1.50u
- S15, S28: footprint ScottoKeebs_Hotswap:Hotswap_Choc_V1_1.25u -> With-Hotswap & Switches:Hotswap_Choc_V1_1.25u
- S41, S42: footprint ScottoKeebs_Hotswap:Hotswap_Choc_V1_1.75u -> With-Hotswap & Switches:Hotswap_Choc_V1_1.75u
- S59, S60: footprint ScottoKeebs_Hotswap:Hotswap_Choc_V1_3.00u -> With-Hotswap & Switches:Hotswap_Choc_V1_3.00u
